Commit message: fix(sim): remove xacro pi redefinition warning

File: ros2_ws/src/tactile_sim/urdf/phase6_arm.urdf.xacro (robot description, xacro)
@@ -1,5 +1,4 @@
 <?xml version="1.0"?>
 <robot name="phase6_arm" xmlns:xacro="http://www.ros.org/wiki/xacro">
-  <xacro:property name="pi" value="3.1415926535897931"/>
   <link name="base_link">
     <inertial>
